File: 78xx/PSU-78xx.sch (KiCad schematic (older format))
At the start: 6 parts

Commit message: Update to KiCad 5
Parts:
- C? (x2): symbol C_Small -> PSU-78xx-rescue:C_Small
- C? (x2): symbol CP1_Small -> PSU-78xx-rescue:CP1_Small
- J?: symbol Conn_01x02 -> PSU-78xx-rescue:Conn_01x02
- U?: symbol L7805 -> PSU-78xx-rescue:L7805
Connections:
- wire segments 13 -> 17
Changed lines of the file:
@@
-EESchema Schematic File Version 2
-LIBS:power
-LIBS:device
-LIBS:transistors
-LIBS:conn
-LIBS:linear
-LIBS:regul
-LIBS:74xx
-LIBS:cmos4000
-LIBS:adc-dac
-LIBS:memory
-LIBS:xilinx
-LIBS:microcontrollers
-LIBS:dsp
-LIBS:microchip
-LIBS:analog_switches
-LIBS:motorola
-LIBS:texas
-LIBS:intel
-LIBS:audio
-LIBS:interface
-LIBS:digital-audio
-LIBS:philips
-LIBS:display
-LIBS:cypress
-LIBS:siliconi
-LIBS:opto
-LIBS:atmel
-LIBS:contrib
-LIBS:valves
-EELAYER 25 0
+EESchema Schematic File Version 4
+LIBS:PSU-78xx-cache
+EELAYER 26 0
 EELAYER END
 $Descr A4 11693 8268
@@
 $EndDescr
 $Comp
-L L7805 U?
+L PSU-78xx-rescue:L7805 U?
 U 1 1 5B2F77C9
 P 5800 3600
@@
 $EndComp
 $Comp
-L C_Small C?
+L PSU-78xx-rescue:C_Small C?
 U 1 1 5B2F7881
 P 5400 3800
@@
 $EndComp
 $Comp
-L CP1_Small C?
+L PSU-78xx-rescue:CP1_Small C?
 U 1 1 5B2F78AD
 P 5200 3800
@@
 $EndComp
 $Comp
-L Conn_01x02 J?
+L PSU-78xx-rescue:Conn_01x02 J?
 U 1 1 5B2F796D
 P 4700 3600
@@
 $EndComp
 $Comp
-L CP1_Small C?
+L PSU-78xx-rescue:CP1_Small C?
 U 1 1 5B2F7D67
 P 6200 3800
@@
 $EndComp
 $Comp
-L C_Small C?
+L PSU-78xx-rescue:C_Small C?
 U 1 1 5B2F7D92
 P 6400 3800
@@
 $EndComp
 $Comp
-L GND #PWR?
+L PSU-78xx-rescue:GND #PWR?
 U 1 1 5B2F7DC4
 P 5200 4000
@@
 $EndComp
 $Comp
-L GND #PWR?
+L PSU-78xx-rescue:GND #PWR?
 U 1 1 5B2F7DE8
 P 5400 4000
@@
 $EndComp
 $Comp
-L GND #PWR?
+L PSU-78xx-rescue:GND #PWR?
 U 1 1 5B2F7E05
 P 5800 4000
@@
 $EndComp
 $Comp
-L GND #PWR?
+L PSU-78xx-rescue:GND #PWR?
 U 1 1 5B2F7E22
 P 6200 4000
@@
 $EndComp
 $Comp
-L GND #PWR?
+L PSU-78xx-rescue:GND #PWR?
 U 1 1 5B2F7E3F
 P 6400 4000
@@
 $EndComp
 $Comp
-L GND #PWR?
+L PSU-78xx-rescue:GND #PWR?
 U 1 1 5B2F7E5C
 P 5000 4000
@@
 $EndComp
 Wire Wire Line
-	4900 3600 5500 3600
+	4900 3600 5200 3600
 Wire Wire Line
 	5200 3600 5200 3700
@@
 Connection ~ 5400 3600
 Wire Wire Line
-	6100 3600 6600 3600
+	6100 3600 6200 3600
 Wire Wire Line
 	6200 3600 6200 3700
@@
 	6400 3900 6400 4000
 Connection ~ 6400 3600
+Wire Wire Line
+	5200 3600 5400 3600
+Wire Wire Line
+	5400 3600 5500 3600
+Wire Wire Line
+	6200 3600 6400 3600
+Wire Wire Line
+	6400 3600 6600 3600
 $EndSCHEMATC
