File: ISP/AVR/2x5/ISP.sch (KiCad schematic (older format))
At the start: 1 part

Commit message: Update to KiCad 5
Parts:
- removed P?: AVR-ISP, symbol CONN_02X05
- added J?: ISP, symbol Connector_Generic:Conn_02x05_Odd_Even
Connections:
- wire segments 11 -> 14
Changed lines of the file:
@@
-EESchema Schematic File Version 2
-LIBS:power
-LIBS:device
-LIBS:transistors
-LIBS:conn
-LIBS:linear
-LIBS:regul
-LIBS:74xx
-LIBS:cmos4000
-LIBS:adc-dac
-LIBS:memory
-LIBS:xilinx
-LIBS:microcontrollers
-LIBS:dsp
-LIBS:microchip
-LIBS:analog_switches
-LIBS:motorola
-LIBS:texas
-LIBS:intel
-LIBS:audio
-LIBS:interface
-LIBS:digital-audio
-LIBS:philips
-LIBS:display
-LIBS:cypress
-LIBS:siliconi
-LIBS:opto
-LIBS:atmel
-LIBS:contrib
-LIBS:valves
+EESchema Schematic File Version 4
 LIBS:ISP-cache
-EELAYER 25 0
+EELAYER 26 0
 EELAYER END
 $Descr A4 11693 8268
 encoding utf-8
 Sheet 1 1
-Title "MIDI-USB Interface"
-Date "2014-04-20"
-Rev "1.6"
-Comp "LOFITECH"
+Title ""
+Date "2018-08-19"
+Rev ""
+Comp ""
 Comment1 ""
 Comment2 ""
@@
 Comment4 ""
 $EndDescr
-$Comp
-L CONN_02X05 P?
-U 1 1 57431EB1
-P 4650 6700
-F 0 "P?" H 4650 7000 50  0000 C CNN
-F 1 "AVR-ISP" H 4650 6400 50  0000 C CNN
-F 2 "" H 4650 5500 50  0000 C CNN
-F 3 "" H 4650 5500 50  0000 C CNN
-	1    4650 6700
-	1    0    0    -1
-$EndComp
-$Comp
-L +5V #PWR?
-U 1 1 5743216D
-P 4950 6400
-F 0 "#PWR?" H 4950 6250 50  0001 C CNN
-F 1 "+5V" H 4950 6540 44  0000 C CNN
-F 2 "" H 4950 6400 50  0000 C CNN
-F 3 "" H 4950 6400 50  0000 C CNN
-	1    4950 6400
-	1    0    0    -1
-$EndComp
-$Comp
-L GND #PWR?
-U 1 1 57432181
-P 4950 7000
-F 0 "#PWR?" H 4950 6750 50  0001 C CNN
-F 1 "GND" H 4950 6850 44  0000 C CNN
-F 2 "" H 4950 7000 50  0000 C CNN
-F 3 "" H 4950 7000 50  0000 C CNN
-	1    4950 7000
-	1    0    0    -1
-$EndComp
 Wire Wire Line
 	4900 6600 4950 6600
 Wire Wire Line
-	4950 6600 4950 7000
+	4950 6600 4950 6700
 Wire Wire Line
 	4900 6700 4950 6700
@@
 SCK
 NoConn ~ 4400 6600
+Wire Wire Line
+	4950 6700 4950 6800
+Wire Wire Line
+	4950 6800 4950 6900
+Wire Wire Line
+	4950 6900 4950 7000
+$Comp
+L power:GND #PWR?
+U 1 1 5B7975F0
+P 4950 7000
+F 0 "#PWR?" H 4950 6750 50  0001 C CNN
+F 1 "GND" H 4955 6827 50  0000 C CNN
+F 2 "" H 4950 7000 50  0001 C CNN
+F 3 "" H 4950 7000 50  0001 C CNN
+	1    4950 7000
+	1    0    0    -1
+$EndComp
+$Comp
+L power:+5V #PWR?
+U 1 1 5B797620
+P 4950 6400
+F 0 "#PWR?" H 4950 6250 50  0001 C CNN
+F 1 "+5V" H 4965 6573 50  0000 C CNN
+F 2 "" H 4950 6400 50  0001 C CNN
+F 3 "" H 4950 6400 50  0001 C CNN
+	1    4950 6400
+	1    0    0    -1
+$EndComp
+$Comp
+L Connector_Generic:Conn_02x05_Odd_Even J?
+U 1 1 5B797706
+P 4600 6700
+F 0 "J?" H 4650 7117 50  0000 C CNN
+F 1 "ISP" H 4650 7026 50  0000 C CNN
+F 2 "" H 4600 6700 50  0001 C CNN
+F 3 "~" H 4600 6700 50  0001 C CNN
+	1    4600 6700
+	1    0    0    -1
+$EndComp
 $EndSCHEMATC
