File: ISP/AVR/TP/ISP.sch (KiCad schematic (older format))
At the start: 6 parts

Commit message: Update to KiCad 5
Parts:
- removed P?: Vcc, Measurement_Points:Measurement_Point_Round-SMD-Pad_Big, symbol CONN_01X01
- removed P?: MOSI, Measurement_Points:Measurement_Point_Round-SMD-Pad_Big, symbol CONN_01X01
- removed P?: MISO, Measurement_Points:Measurement_Point_Round-SMD-Pad_Big, symbol CONN_01X01
- removed P?: SCK, Measurement_Points:Measurement_Point_Round-SMD-Pad_Big, symbol CONN_01X01
- removed P?: ~RST, Measurement_Points:Measurement_Point_Round-SMD-Pad_Big, symbol CONN_01X01
- removed P?: GND, Measurement_Points:Measurement_Point_Round-SMD-Pad_Big, symbol CONN_01X01
- added J?: Vcc, symbol Connector_Generic:Conn_01x01
- added J?: MOSI, symbol Connector_Generic:Conn_01x01
- added J?: MISO, symbol Connector_Generic:Conn_01x01
- added J?: SCK, symbol Connector_Generic:Conn_01x01
- added J?: ~RST, symbol Connector_Generic:Conn_01x01
- added J?: GND, symbol Connector_Generic:Conn_01x01
Changed lines of the file:
@@
-EESchema Schematic File Version 2
-LIBS:power
-LIBS:device
-LIBS:transistors
-LIBS:conn
-LIBS:linear
-LIBS:regul
-LIBS:74xx
-LIBS:cmos4000
-LIBS:adc-dac
-LIBS:memory
-LIBS:xilinx
-LIBS:microcontrollers
-LIBS:dsp
-LIBS:microchip
-LIBS:analog_switches
-LIBS:motorola
-LIBS:texas
-LIBS:intel
-LIBS:audio
-LIBS:interface
-LIBS:digital-audio
-LIBS:philips
-LIBS:display
-LIBS:cypress
-LIBS:siliconi
-LIBS:opto
-LIBS:atmel
-LIBS:contrib
-LIBS:valves
-LIBS:ISP-cache
-EELAYER 25 0
+EESchema Schematic File Version 4
+EELAYER 26 0
 EELAYER END
 $Descr A4 11693 8268
 encoding utf-8
 Sheet 1 1
-Title "MIDI-USB Interface"
-Date "2014-04-20"
-Rev "1.6"
-Comp "LOFITECH"
+Title ""
+Date "2018-08-19"
+Rev ""
+Comp ""
 Comment1 ""
 Comment2 ""
@@
 Comment4 ""
 $EndDescr
-$Comp
-L CONN_01X01 P?
-U 1 1 5982C575
-P 6000 6500
-F 0 "P?" H 6000 6600 50  0001 C CNN
-F 1 "Vcc" H 6075 6500 44  0000 L CNN
-F 2 "Measurement_Points:Measurement_Point_Round-SMD-Pad_Big" H 6000 6500 50  0001 C CNN
-F 3 "" H 6000 6500 50  0000 C CNN
-	1    6000 6500
-	1    0    0    -1
-$EndComp
-$Comp
-L CONN_01X01 P?
-U 1 1 5982C5B9
-P 6000 6650
-F 0 "P?" H 6000 6750 50  0001 C CNN
-F 1 "MOSI" H 6075 6650 44  0000 L CNN
-F 2 "Measurement_Points:Measurement_Point_Round-SMD-Pad_Big" H 6000 6650 50  0001 C CNN
-F 3 "" H 6000 6650 50  0000 C CNN
-	1    6000 6650
-	1    0    0    -1
-$EndComp
-$Comp
-L CONN_01X01 P?
-U 1 1 5982C633
-P 6000 6800
-F 0 "P?" H 6000 6900 50  0001 C CNN
-F 1 "MISO" H 6075 6800 44  0000 L CNN
-F 2 "Measurement_Points:Measurement_Point_Round-SMD-Pad_Big" H 6000 6800 50  0001 C CNN
-F 3 "" H 6000 6800 50  0000 C CNN
-	1    6000 6800
-	1    0    0    -1
-$EndComp
-$Comp
-L CONN_01X01 P?
-U 1 1 5982C647
-P 6000 6950
-F 0 "P?" H 6000 7050 50  0001 C CNN
-F 1 "SCK" H 6075 6950 44  0000 L CNN
-F 2 "Measurement_Points:Measurement_Point_Round-SMD-Pad_Big" H 6000 6950 50  0001 C CNN
-F 3 "" H 6000 6950 50  0000 C CNN
-	1    6000 6950
-	1    0    0    -1
-$EndComp
-$Comp
-L CONN_01X01 P?
-U 1 1 5982C65B
-P 6000 7100
-F 0 "P?" H 6000 7200 50  0001 C CNN
-F 1 "~RST" H 6075 7100 44  0000 L CNN
-F 2 "Measurement_Points:Measurement_Point_Round-SMD-Pad_Big" H 6000 7100 50  0001 C CNN
-F 3 "" H 6000 7100 50  0000 C CNN
-	1    6000 7100
-	1    0    0    -1
-$EndComp
-$Comp
-L CONN_01X01 P?
-U 1 1 5982C66F
-P 6000 7250
-F 0 "P?" H 6000 7350 50  0001 C CNN
-F 1 "GND" H 6075 7250 44  0000 L CNN
-F 2 "Measurement_Points:Measurement_Point_Round-SMD-Pad_Big" H 6000 7250 50  0001 C CNN
-F 3 "" H 6000 7250 50  0000 C CNN
-	1    6000 7250
-	1    0    0    -1
-$EndComp
-$Comp
-L +5V #PWR?
-U 1 1 5982C6DB
-P 5700 6400
-F 0 "#PWR?" H 5700 6250 44  0001 C CNN
-F 1 "+5V" H 5700 6540 50  0000 C CNN
-F 2 "" H 5700 6400 50  0000 C CNN
-F 3 "" H 5700 6400 50  0000 C CNN
-	1    5700 6400
-	1    0    0    -1
-$EndComp
-$Comp
-L GND #PWR?
-U 1 1 5982C6EF
-P 5700 7350
-F 0 "#PWR?" H 5700 7100 50  0001 C CNN
-F 1 "GND" H 5700 7200 50  0000 C CNN
-F 2 "" H 5700 7350 50  0000 C CNN
-F 3 "" H 5700 7350 50  0000 C CNN
-	1    5700 7350
-	1    0    0    -1
-$EndComp
 Wire Wire Line
 	5700 7350 5700 7250
@@
 Wire Wire Line
 	5550 7100 5800 7100
+$Comp
+L power:GND #PWR?
+U 1 1 5B7975F0
+P 5700 7350
+F 0 "#PWR?" H 5700 7100 50  0001 C CNN
+F 1 "GND" H 5705 7177 50  0000 C CNN
+F 2 "" H 5700 7350 50  0001 C CNN
+F 3 "" H 5700 7350 50  0001 C CNN
+	1    5700 7350
+	1    0    0    -1
+$EndComp
+$Comp
+L power:+5V #PWR?
+U 1 1 5B797620
+P 5700 6400
+F 0 "#PWR?" H 5700 6250 50  0001 C CNN
+F 1 "+5V" H 5715 6573 50  0000 C CNN
+F 2 "" H 5700 6400 50  0001 C CNN
+F 3 "" H 5700 6400 50  0001 C CNN
+	1    5700 6400
+	1    0    0    -1
+$EndComp
+$Comp
+L Connector_Generic:Conn_01x01 J?
+U 1 1 5B7976D8
+P 6000 6500
+F 0 "J?" H 6080 6542 50  0001 L CNN
+F 1 "Vcc" H 6075 6500 50  0000 L CNN
+F 2 "" H 6000 6500 50  0001 C CNN
+F 3 "~" H 6000 6500 50  0001 C CNN
+	1    6000 6500
+	1    0    0    -1
+$EndComp
+$Comp
+L Connector_Generic:Conn_01x01 J?
+U 1 1 5B797758
+P 6000 6650
+F 0 "J?" H 6080 6692 50  0001 L CNN
+F 1 "MOSI" H 6075 6650 50  0000 L CNN
+F 2 "" H 6000 6650 50  0001 C CNN
+F 3 "~" H 6000 6650 50  0001 C CNN
+	1    6000 6650
+	1    0    0    -1
+$EndComp
+$Comp
+L Connector_Generic:Conn_01x01 J?
+U 1 1 5B797784
+P 6000 6800
+F 0 "J?" H 6080 6842 50  0001 L CNN
+F 1 "MISO" H 6075 6800 50  0000 L CNN
+F 2 "" H 6000 6800 50  0001 C CNN
+F 3 "~" H 6000 6800 50  0001 C CNN
+	1    6000 6800
+	1    0    0    -1
+$EndComp
+$Comp
+L Connector_Generic:Conn_01x01 J?
+U 1 1 5B7977D1
+P 6000 6950
+F 0 "J?" H 6080 6992 50  0001 L CNN
+F 1 "SCK" H 6075 6950 50  0000 L CNN
+F 2 "" H 6000 6950 50  0001 C CNN
+F 3 "~" H 6000 6950 50  0001 C CNN
+	1    6000 6950
+	1    0    0    -1
+$EndComp
+$Comp
+L Connector_Generic:Conn_01x01 J?
+U 1 1 5B79782B
+P 6000 7100
+F 0 "J?" H 6080 7142 50  0001 L CNN
+F 1 "~RST" H 6075 7100 50  0000 L CNN
+F 2 "" H 6000 7100 50  0001 C CNN
+F 3 "~" H 6000 7100 50  0001 C CNN
+	1    6000 7100
+	1    0    0    -1
+$EndComp
+$Comp
+L Connector_Generic:Conn_01x01 J?
+U 1 1 5B79789E
+P 6000 7250
+F 0 "J?" H 6080 7292 50  0001 L CNN
+F 1 "GND" H 6075 7250 50  0000 L CNN
+F 2 "" H 6000 7250 50  0001 C CNN
+F 3 "~" H 6000 7250 50  0001 C CNN
+	1    6000 7250
+	1    0    0    -1
+$EndComp
 $EndSCHEMATC
