File: ISP/STM32/4x1/ISP.sch (KiCad schematic (older format))
At the start: 1 part

Commit message: Update to KiCad 5
Parts:
- removed P?: JTAG, symbol CONN_01X04
- added J?: ISP, symbol Connector_Generic:Conn_01x04
Changed lines of the file:
@@
-EESchema Schematic File Version 2
-LIBS:power
-LIBS:device
-LIBS:transistors
-LIBS:conn
-LIBS:linear
-LIBS:regul
-LIBS:74xx
-LIBS:cmos4000
-LIBS:adc-dac
-LIBS:memory
-LIBS:xilinx
-LIBS:microcontrollers
-LIBS:dsp
-LIBS:microchip
-LIBS:analog_switches
-LIBS:motorola
-LIBS:texas
-LIBS:intel
-LIBS:audio
-LIBS:interface
-LIBS:digital-audio
-LIBS:philips
-LIBS:display
-LIBS:cypress
-LIBS:siliconi
-LIBS:opto
-LIBS:atmel
-LIBS:contrib
-LIBS:valves
-LIBS:ISP-cache
-EELAYER 25 0
+EESchema Schematic File Version 4
+EELAYER 26 0
 EELAYER END
 $Descr A4 11693 8268
 encoding utf-8
 Sheet 1 1
-Title "MIDI-USB Interface"
-Date "2014-04-20"
-Rev "1.6"
-Comp "LOFITECH"
+Title ""
+Date "2018-08-19"
+Rev ""
+Comp ""
 Comment1 ""
 Comment2 ""
@@
 Comment4 ""
 $EndDescr
-$Comp
-L CONN_01X04 P?
-U 1 1 57431ECA
-P 1850 6750
-F 0 "P?" H 1850 7000 50  0000 C CNN
-F 1 "JTAG" V 1950 6750 50  0000 C CNN
-F 2 "" H 1850 6750 50  0000 C CNN
-F 3 "" H 1850 6750 50  0000 C CNN
-	1    1850 6750
-	1    0    0    -1
-$EndComp
 Wire Wire Line
 	1650 6700 1450 6700
@@
 Wire Wire Line
 	1600 6900 1650 6900
-$Comp
-L GND #PWR?
-U 1 1 57432559
-P 1600 7000
-F 0 "#PWR?" H 1600 6750 44  0001 C CNN
-F 1 "GND" H 1600 6850 50  0000 C CNN
-F 2 "" H 1600 7000 50  0000 C CNN
-F 3 "" H 1600 7000 50  0000 C CNN
-	1    1600 7000
-	1    0    0    -1
-$EndComp
 Wire Wire Line
 	1650 6600 1600 6600
@@
 	1600 6600 1600 6500
 $Comp
-L +3V3 #PWR?
-U 1 1 5743258D
+L power:GND #PWR?
+U 1 1 5B79771B
+P 1600 7000
+F 0 "#PWR?" H 1600 6750 50  0001 C CNN
+F 1 "GND" H 1605 6827 50  0000 C CNN
+F 2 "" H 1600 7000 50  0001 C CNN
+F 3 "" H 1600 7000 50  0001 C CNN
+	1    1600 7000
+	1    0    0    -1
+$EndComp
+$Comp
+L Connector_Generic:Conn_01x04 J?
+U 1 1 5B7977FD
+P 1850 6700
+F 0 "J?" H 1930 6692 50  0000 L CNN
+F 1 "ISP" H 1930 6601 50  0000 L CNN
+F 2 "" H 1850 6700 50  0001 C CNN
+F 3 "~" H 1850 6700 50  0001 C CNN
+	1    1850 6700
+	1    0    0    -1
+$EndComp
+$Comp
+L power:+3V3 #PWR?
+U 1 1 5B797864
 P 1600 6500
-F 0 "#PWR?" H 1600 6350 44  0001 C CNN
-F 1 "+3V3" H 1600 6640 50  0000 C CNN
-F 2 "" H 1600 6500 50  0000 C CNN
-F 3 "" H 1600 6500 50  0000 C CNN
+F 0 "#PWR?" H 1600 6350 50  0001 C CNN
+F 1 "+3V3" H 1615 6673 50  0000 C CNN
+F 2 "" H 1600 6500 50  0001 C CNN
+F 3 "" H 1600 6500 50  0001 C CNN
 	1    1600 6500
 	1    0    0    -1
