File: Discovery-F4/Discovery-F4 base board.sch (KiCad schematic (older format))
At the start: 4 parts, among them P1 P1, P2 P2, P3 JP3, P4 JP2

Commit message: Update to KiCad 5
Parts:
- P1, P2: symbol CONN_02X25 -> Discovery-F4-base-board-rescue:CONN_02X25
- P3, P4: symbol CONN_01X02 -> Discovery-F4-base-board-rescue:CONN_01X02
Changed lines of the file:
@@
-EESchema Schematic File Version 2
-LIBS:power
-LIBS:device
-LIBS:transistors
-LIBS:conn
-LIBS:linear
-LIBS:regul
-LIBS:74xx
-LIBS:cmos4000
-LIBS:adc-dac
-LIBS:memory
-LIBS:xilinx
-LIBS:microcontrollers
-LIBS:dsp
-LIBS:microchip
-LIBS:analog_switches
-LIBS:motorola
-LIBS:texas
-LIBS:intel
-LIBS:audio
-LIBS:interface
-LIBS:digital-audio
-LIBS:philips
-LIBS:display
-LIBS:cypress
-LIBS:siliconi
-LIBS:opto
-LIBS:atmel
-LIBS:contrib
-LIBS:valves
+EESchema Schematic File Version 4
 LIBS:Discovery-F4 base board-cache
-EELAYER 25 0
+EELAYER 26 0
 EELAYER END
 $Descr A4 11693 8268
@@
 $EndDescr
 $Comp
-L CONN_02X25 P1
+L Discovery-F4-base-board-rescue:CONN_02X25 P1
 U 1 1 5749427D
 P 3850 3600
@@
 $EndComp
 $Comp
-L CONN_01X02 P3
+L Discovery-F4-base-board-rescue:CONN_01X02 P3
 U 1 1 5749430F
 P 8400 2450
@@
 $EndComp
 $Comp
-L CONN_01X02 P4
+L Discovery-F4-base-board-rescue:CONN_01X02 P4
 U 1 1 57494354
 P 8400 3200
@@
 $EndComp
 $Comp
-L GND #PWR01
+L power:GND #PWR01
 U 1 1 5749437C
 P 8100 2600
@@
 $EndComp
 $Comp
-L GND #PWR02
+L power:GND #PWR02
 U 1 1 5749439A
 P 8100 3350
@@
 $EndComp
 Wire Wire Line
-	8100 2600 8100 2400
+	8100 2600 8100 2500
 Wire Wire Line
 	8100 2400 8200 2400
@@
 	8200 3150 8100 3150
 Wire Wire Line
-	8100 3150 8100 3350
+	8100 3150 8100 3250
 Wire Wire Line
 	8200 3250 8100 3250
@@
 	4500 4600 4100 4600
 $Comp
-L CONN_02X25 P2
+L Discovery-F4-base-board-rescue:CONN_02X25 P2
 U 1 1 57494C92
 P 6450 3600
@@
 	3600 2400 3500 2400
 Wire Wire Line
-	3500 2400 3500 4900
+	3500 2400 3500 4800
 Wire Wire Line
 	3600 4800 3500 4800
@@
 	4100 2400 4200 2400
 Wire Wire Line
-	4200 2400 4200 4900
+	4200 2400 4200 4800
 Wire Wire Line
 	4200 4800 4100 4800
 Connection ~ 4200 4800
 $Comp
-L GND #PWR03
+L power:GND #PWR03
 U 1 1 574953E5
 P 3500 4900
@@
 $EndComp
 $Comp
-L GND #PWR04
+L power:GND #PWR04
 U 1 1 5749542E
 P 4200 4900
@@
 	6200 2400 6100 2400
 Wire Wire Line
-	6100 2400 6100 4900
+	6100 2400 6100 4800
 Connection ~ 6100 4800
 Wire Wire Line
 	6700 2400 6800 2400
 Wire Wire Line
-	6800 2400 6800 4900
+	6800 2400 6800 4800
 Connection ~ 6800 4800
 $Comp
-L GND #PWR05
+L power:GND #PWR05
 U 1 1 574955E7
 P 6100 4900
@@
 $EndComp
 $Comp
-L GND #PWR06
+L power:GND #PWR06
 U 1 1 574955FE
 P 6800 4900
@@
 Text Label 7100 4700 2    44   ~ 0
 PC7
+Wire Wire Line
+	8100 2500 8100 2400
+Wire Wire Line
+	8100 3250 8100 3350
+Wire Wire Line
+	3500 4800 3500 4900
+Wire Wire Line
+	4200 4800 4200 4900
+Wire Wire Line
+	6100 4800 6100 4900
+Wire Wire Line
+	6800 4800 6800 4900
 $EndSCHEMATC

Commit message: Update to KiCad 5.1.7
Parts:
- P1, P2: symbol Discovery-F4-base-board-rescue:CONN_02X25 -> Discovery-F4-base-board-rescue:CONN_02X25-Discovery-F4-base-board-rescue
- P3, P4: symbol Discovery-F4-base-board-rescue:CONN_01X02 -> Discovery-F4-base-board-rescue:CONN_01X02-Discovery-F4-base-board-rescue
Changed lines of the file:
@@
 EESchema Schematic File Version 4
-LIBS:Discovery-F4 base board-cache
-EELAYER 26 0
+EELAYER 30 0
 EELAYER END
 $Descr A4 11693 8268
@@
 $EndDescr
 $Comp
-L Discovery-F4-base-board-rescue:CONN_02X25 P1
+L Discovery-F4-base-board-rescue:CONN_02X25-Discovery-F4-base-board-rescue P1
 U 1 1 5749427D
 P 3850 3600
@@
 $EndComp
 $Comp
-L Discovery-F4-base-board-rescue:CONN_01X02 P3
+L Discovery-F4-base-board-rescue:CONN_01X02-Discovery-F4-base-board-rescue P3
 U 1 1 5749430F
 P 8400 2450
@@
 $EndComp
 $Comp
-L Discovery-F4-base-board-rescue:CONN_01X02 P4
+L Discovery-F4-base-board-rescue:CONN_01X02-Discovery-F4-base-board-rescue P4
 U 1 1 57494354
 P 8400 3200
@@
 	4500 4600 4100 4600
 $Comp
-L Discovery-F4-base-board-rescue:CONN_02X25 P2
+L Discovery-F4-base-board-rescue:CONN_02X25-Discovery-F4-base-board-rescue P2
 U 1 1 57494C92
 P 6450 3600
