File: PSUs/78xx/PSU-78xx.sch (KiCad schematic (older format))
At the start: 6 parts

Commit message: Update to KiCad 5.1.7
Parts:
- C? (x2): symbol PSU-78xx-rescue:C_Small -> PSU-78xx-rescue:C_Small-PSU-78xx-rescue
- C? (x2): symbol PSU-78xx-rescue:CP1_Small -> PSU-78xx-rescue:CP1_Small-PSU-78xx-rescue
- J?: symbol PSU-78xx-rescue:Conn_01x02 -> PSU-78xx-rescue:Conn_01x02-PSU-78xx-rescue
- U?: symbol PSU-78xx-rescue:L7805 -> PSU-78xx-rescue:L7805-PSU-78xx-rescue
Changed lines of the file:
@@
 EESchema Schematic File Version 4
-LIBS:PSU-78xx-cache
-EELAYER 26 0
+EELAYER 30 0
 EELAYER END
 $Descr A4 11693 8268
@@
 $EndDescr
 $Comp
-L PSU-78xx-rescue:L7805 U?
+L PSU-78xx-rescue:L7805-PSU-78xx-rescue U?
 U 1 1 5B2F77C9
 P 5800 3600
@@
 $EndComp
 $Comp
-L PSU-78xx-rescue:C_Small C?
+L PSU-78xx-rescue:C_Small-PSU-78xx-rescue C?
 U 1 1 5B2F7881
 P 5400 3800
@@
 $EndComp
 $Comp
-L PSU-78xx-rescue:CP1_Small C?
+L PSU-78xx-rescue:CP1_Small-PSU-78xx-rescue C?
 U 1 1 5B2F78AD
 P 5200 3800
@@
 $EndComp
 $Comp
-L PSU-78xx-rescue:Conn_01x02 J?
+L PSU-78xx-rescue:Conn_01x02-PSU-78xx-rescue J?
 U 1 1 5B2F796D
 P 4700 3600
@@
 $EndComp
 $Comp
-L PSU-78xx-rescue:CP1_Small C?
+L PSU-78xx-rescue:CP1_Small-PSU-78xx-rescue C?
 U 1 1 5B2F7D67
 P 6200 3800
@@
 $EndComp
 $Comp
-L PSU-78xx-rescue:C_Small C?
+L PSU-78xx-rescue:C_Small-PSU-78xx-rescue C?
 U 1 1 5B2F7D92
 P 6400 3800
@@
 $EndComp
 $Comp
-L PSU-78xx-rescue:GND #PWR?
+L PSU-78xx-rescue:GND-PSU-78xx-rescue #PWR?
 U 1 1 5B2F7DC4
 P 5200 4000
@@
 $EndComp
 $Comp
-L PSU-78xx-rescue:GND #PWR?
+L PSU-78xx-rescue:GND-PSU-78xx-rescue #PWR?
 U 1 1 5B2F7DE8
 P 5400 4000
@@
 $EndComp
 $Comp
-L PSU-78xx-rescue:GND #PWR?
+L PSU-78xx-rescue:GND-PSU-78xx-rescue #PWR?
 U 1 1 5B2F7E05
 P 5800 4000
@@
 $EndComp
 $Comp
-L PSU-78xx-rescue:GND #PWR?
+L PSU-78xx-rescue:GND-PSU-78xx-rescue #PWR?
 U 1 1 5B2F7E22
 P 6200 4000
@@
 $EndComp
 $Comp
-L PSU-78xx-rescue:GND #PWR?
+L PSU-78xx-rescue:GND-PSU-78xx-rescue #PWR?
 U 1 1 5B2F7E3F
 P 6400 4000
@@
 $EndComp
 $Comp
-L PSU-78xx-rescue:GND #PWR?
+L PSU-78xx-rescue:GND-PSU-78xx-rescue #PWR?
 U 1 1 5B2F7E5C
 P 5000 4000
