File: STM32/Discovery-F4/Discovery-F4 base board.kicad_sch (KiCad schematic)
At the start: 4 parts, among them P1 P1, P2 P2, P3 JP3, P4 JP2

Commit message: Fix grid alignment and update to KiCad 9
Parts:
- removed P1: P1, Pin_Headers:Pin_Header_Straight_2x25, symbol Discovery-F4-base-board-rescue:CONN_02X25-Discovery-F4-base-board-rescue
- removed P2: P2, Pin_Headers:Pin_Header_Straight_2x25, symbol Discovery-F4-base-board-rescue:CONN_02X25-Discovery-F4-base-board-rescue
- removed P3: JP3, Pin_Headers:Pin_Header_Straight_1x02, symbol Discovery-F4-base-board-rescue:CONN_01X02-Discovery-F4-base-board-rescue
- removed P4: JP2, Pin_Headers:Pin_Header_Straight_1x02, symbol Discovery-F4-base-board-rescue:CONN_01X02-Discovery-F4-base-board-rescue
- added J1, J2: Conn_01x02, symbol Connector_Generic:Conn_01x02
- added J3, J4: Conn_02x25_Odd_Even, symbol Connector_Generic:Conn_02x25_Odd_Even
Connections:
- net 3V: now also J4.5 (Pin_5), J4.6 (Pin_6)
- net 5V: now also J4.3 (Pin_3), J4.4 (Pin_4)
- net BOOT0: now also J4.21 (Pin_21)
- net GND: now also J1.1 (Pin_1), J1.2 (Pin_2), J2.1 (Pin_1), J2.2 (Pin_2), J3.1 (Pin_1), J3.2 (Pin_2), J3.23 (Pin_23), J3.49 (Pin_49), J3.5 (Pin_5), J3.50 (Pin_50), J4.1 (Pin_1), J4.2 (Pin_2), J4.49 (Pin_49), J4.50 (Pin_50)
- net NRST: now also J3.6 (Pin_6)
- net PA0: now also J3.12 (Pin_12)
- net PA1: now also J3.11 (Pin_11)
- net PA10: now also J4.41 (Pin_41)
- net PA13: now also J4.42 (Pin_42)
- net PA14: now also J4.39 (Pin_39)
- net PA15: now also J4.40 (Pin_40)
- net PA2: now also J3.14 (Pin_14)
- net PA3: now also J3.13 (Pin_13)
- net PA4: now also J3.16 (Pin_16)
- net PA5: now also J3.15 (Pin_15)
- net PA6: now also J3.18 (Pin_18)
- net PA7: now also J3.17 (Pin_17)
- net PA8: now also J4.43 (Pin_43)
- net PA9: now also J4.44 (Pin_44)
- net PB0: now also J3.22 (Pin_22)
- net PB1: now also J3.21 (Pin_21)
- net PB10: now also J3.34 (Pin_34)
- net PB11: now also J3.35 (Pin_35)
- net PB12: now also J3.36 (Pin_36)
- net PB13: now also J3.37 (Pin_37)
- net PB14: now also J3.38 (Pin_38)
- net PB15: now also J3.39 (Pin_39)
- net PB2: now also J3.24 (Pin_24)
- net PB3: now also J4.28 (Pin_28)
- net PB4: now also J4.25 (Pin_25)
- net PB5: now also J4.26 (Pin_26)
- net PB6: now also J4.23 (Pin_23)
- net PB7: now also J4.24 (Pin_24)
- net PB8: now also J4.19 (Pin_19)
- net PB9: now also J4.18 (Pin_18)
- net PC0: now also J3.8 (Pin_8)
- net PC1: now also J3.7 (Pin_7)
- net PC10: now also J4.37 (Pin_37)
- net PC11: now also J4.38 (Pin_38)
- net PC12: now also J4.35 (Pin_35)
- net PC13: now also J4.12 (Pin_12)
- net PC14: now also J4.9 (Pin_9)
- net PC15: now also J4.10 (Pin_10)
- net PC2: now also J3.10 (Pin_10)
- net PC3: now also J3.9 (Pin_9)
- net PC4: now also J3.20 (Pin_20)
- net PC5: now also J3.19 (Pin_19)
- net PC6: now also J4.47 (Pin_47)
- net PC7: now also J4.48 (Pin_48)
- net PC8: now also J4.45 (Pin_45)
- net PC9: now also J4.46 (Pin_46)
- net PD0: now also J4.36 (Pin_36)
- net PD1: now also J4.33 (Pin_33)
- net PD10: now also J3.42 (Pin_42)
- net PD11: now also J3.43 (Pin_43)
- net PD12: now also J3.44 (Pin_44)
- net PD13: now also J3.45 (Pin_45)
- net PD14: now also J3.46 (Pin_46)
- net PD15: now also J3.47 (Pin_47)
- net PD2: now also J4.34 (Pin_34)
- net PD3: now also J4.31 (Pin_31)
- net PD4: now also J4.32 (Pin_32)
- net PD5: now also J4.29 (Pin_29)
- net PD6: now also J4.30 (Pin_30)
- net PD7: now also J4.27 (Pin_27)
- net PD8: now also J3.40 (Pin_40)
- net PD9: now also J3.41 (Pin_41)
- net PE0: now also J4.17 (Pin_17)
- net PE1: now also J4.20 (Pin_20)
- net PE10: now also J3.28 (Pin_28)
- net PE11: now also J3.29 (Pin_29)
- net PE12: now also J3.30 (Pin_30)
- net PE13: now also J3.31 (Pin_31)
- net PE14: now also J3.32 (Pin_32)
- net PE15: now also J3.33 (Pin_33)
- net PE2: now also J4.15 (Pin_15)
- net PE3: now also J4.16 (Pin_16)
- net PE4: now also J4.13 (Pin_13)
- net PE5: now also J4.14 (Pin_14)
- net PE6: now also J4.11 (Pin_11)
- net PE7: now also J3.25 (Pin_25)
- net PE8: now also J3.26 (Pin_26)
- net PE9: now also J3.27 (Pin_27)
- net PH0: now also J4.7 (Pin_7)
- net PH1: now also J4.8 (Pin_8)
- net VDD: now also J3.3 (Pin_3), J3.4 (Pin_4), J4.22 (Pin_22)
